Commit message: actualizar

File: src/mi_robot_mecanum/urdf/mi_robot.urdf.xacro (robot description, xacro)
@@ -107,5 +107,5 @@
         <scan>
           <horizontal>
-            <samples>1600</samples>
+            <samples>2000</samples>
             <resolution>1</resolution>
             <min_angle>-3.14159265</min_angle>
@@ -114,6 +114,6 @@
         </scan>
         <range>
-          <min>0.15</min>
-          <max>25.0</max>
+          <min>0.2</min>
+          <max>20.0</max>
           <resolution>0.01</resolution>
           <noise>
@@ -156,10 +156,10 @@
   <gazebo reference="camara_link">
     <sensor name="astra" type="rgbd_camera">
-      <topic>/camara</topic>
+      <topic>/camera</topic>
       <gz_frame_id>camara_link</gz_frame_id>
       <update_rate>30</update_rate>
       <always_on>1</always_on>
       <camera>
-        <horizontal_fov>1.57079632679</horizontal_fov>   <!-- 90° -->
+        <horizontal_fov>1.01927</horizontal_fov>   <!-- 58.4° -->
         <image>
           <width>640</width>
@@ -168,11 +168,11 @@
         </image>
         <clip>
-          <near>0.1</near>
-          <far>8.0</far>
+          <near>0.4</near>
+          <far>2.0</far>
         </clip>
         <depth_camera>
           <clip>
-            <near>0.1</near>
-            <far>8.0</far>
+            <near>0.4</near>
+            <far>2.0</far>
           </clip>
         </depth_camera>
@@ -181,18 +181,18 @@
   </gazebo>
   <!-- ===================== Plugins de Gazebo (Parte 1) ===================== -->
-  <!-- Motor de una rueda: recibe ω (rad/s) en /vel_rueda_<prefijo>.
+  <!-- Motor de una rueda: recibe ω (rad/s) en /<corto>_wheel_cmd_vel.
        No se usa MecanumDrive: la cinemática la escriben ustedes en el nodo cinematica. -->
-  <xacro:macro name="motor" params="prefijo">
+  <xacro:macro name="motor" params="prefijo corto">
     <plugin filename="gz-sim-joint-controller-system" name="gz::sim::systems::JointController">
       <joint_name>joint_rueda_${prefijo}</joint_name>
       <use_force_commands>false</use_force_commands>
-      <topic>/vel_rueda_${prefijo}</topic>
+      <topic>/${corto}_wheel_cmd_vel</topic>
     </plugin>
   </xacro:macro>
   <gazebo>
-    <xacro:motor prefijo="del_izq"/>
-    <xacro:motor prefijo="del_der"/>
-    <xacro:motor prefijo="tra_izq"/>
-    <xacro:motor prefijo="tra_der"/>
+    <xacro:motor prefijo="del_izq" corto="fl"/>
+    <xacro:motor prefijo="del_der" corto="fr"/>
+    <xacro:motor prefijo="tra_izq" corto="rl"/>
+    <xacro:motor prefijo="tra_der" corto="rr"/>
     <plugin filename="gz-sim-joint-state-publisher-system" name="gz::sim::systems::JointStatePublisher"/>
   </gazebo>

Commit message: actualizar

File: src/mi_robot_mecanum/urdf/mi_robot.urdf.xacro (robot description, xacro)
@@ -127,35 +127,35 @@
   </gazebo>
   <!-- ===================== Orbbec Astra (Parte 2) ===================== -->
-  <link name="camara_link">
+  <link name="camera_link">
     <visual>
       <origin xyz="0 0 0" rpy="0 0 0"/>
-      <geometry><box size="0.04 0.165 0.048"/></geometry>
+      <geometry><box size="0.03 0.165 0.04"/></geometry>
       <material name="negro_camara"><color rgba="0.1 0.1 0.1 1"/></material>
     </visual>
     <collision>
       <origin xyz="0 0 0" rpy="0 0 0"/>
-      <geometry><box size="0.04 0.165 0.048"/></geometry>
+      <geometry><box size="0.03 0.165 0.04"/></geometry>
     </collision>
     <inertial>
       <origin xyz="0 0 0" rpy="0 0 0"/>
       <mass value="0.31"/>
-      <xacro:inercia_caja m="0.31" x="0.04" y="0.165" z="0.048"/>
+      <xacro:inercia_caja m="0.31" x="0.03" y="0.165" z="0.04"/>
     </inertial>
   </link>
   <joint name="joint_camara" type="fixed">
     <parent link="base_link"/>
-    <child link="camara_link"/>
+    <child link="camera_link"/>
     <origin xyz="0.16 0 0.09" rpy="0 0 0"/>
   </joint>
-  <link name="camara_optica_link"/>
+  <link name="camera_optical_link"/>
   <joint name="joint_camara_optica" type="fixed">
-    <parent link="camara_link"/>
-    <child link="camara_optica_link"/>
+    <parent link="camera_link"/>
+    <child link="camera_optical_link"/>
     <origin xyz="0 0 0" rpy="-${pi/2} 0 -${pi/2}"/>
   </joint>
-  <gazebo reference="camara_link">
+  <gazebo reference="camera_link">
     <sensor name="astra" type="rgbd_camera">
       <topic>/camera</topic>
-      <gz_frame_id>camara_link</gz_frame_id>
+      <gz_frame_id>camera_link</gz_frame_id>
       <update_rate>30</update_rate>
       <always_on>1</always_on>

Commit message: actualizar

File: src/mi_robot_mecanum/urdf/mi_robot.urdf.xacro (robot description, xacro)
@@ -127,5 +127,5 @@
   </gazebo>
   <!-- ===================== Orbbec Astra (Parte 2) ===================== -->
-  <link name="camera_link">
+  <link name="camara_link">
     <visual>
       <origin xyz="0 0 0" rpy="0 0 0"/>
@@ -145,21 +145,21 @@
   <joint name="joint_camara" type="fixed">
     <parent link="base_link"/>
-    <child link="camera_link"/>
+    <child link="camara_link"/>
     <origin xyz="0.16 0 0.09" rpy="0 0 0"/>
   </joint>
-  <link name="camera_optical_link"/>
+  <link name="camara_optica_link"/>
   <joint name="joint_camara_optica" type="fixed">
-    <parent link="camera_link"/>
-    <child link="camera_optical_link"/>
+    <parent link="camara_link"/>
+    <child link="camara_optica_link"/>
     <origin xyz="0 0 0" rpy="-${pi/2} 0 -${pi/2}"/>
   </joint>
-  <gazebo reference="camera_link">
+  <gazebo reference="camara_link">
     <sensor name="astra" type="rgbd_camera">
-      <topic>/camera</topic>
-      <gz_frame_id>camera_link</gz_frame_id>
+      <topic>/camara</topic>
+      <gz_frame_id>camara_link</gz_frame_id>
       <update_rate>30</update_rate>
       <always_on>1</always_on>
       <camera>
-        <horizontal_fov>1.01927</horizontal_fov>   <!-- 58.4° -->
+        <horizontal_fov>1.01927</horizontal_fov>   <!-- en radianes -->
         <image>
           <width>640</width>
@@ -181,18 +181,18 @@
   </gazebo>
   <!-- ===================== Plugins de Gazebo (Parte 1) ===================== -->
-  <!-- Motor de una rueda: recibe ω (rad/s) en /<corto>_wheel_cmd_vel.
+  <!-- Motor de una rueda: recibe ω (rad/s) en /vel_rueda_<prefijo>.
        No se usa MecanumDrive: la cinemática la escriben ustedes en el nodo cinematica. -->
-  <xacro:macro name="motor" params="prefijo corto">
+  <xacro:macro name="motor" params="prefijo">
     <plugin filename="gz-sim-joint-controller-system" name="gz::sim::systems::JointController">
       <joint_name>joint_rueda_${prefijo}</joint_name>
       <use_force_commands>false</use_force_commands>
-      <topic>/${corto}_wheel_cmd_vel</topic>
+      <topic>/vel_rueda_${prefijo}</topic>
     </plugin>
   </xacro:macro>
   <gazebo>
-    <xacro:motor prefijo="del_izq" corto="fl"/>
-    <xacro:motor prefijo="del_der" corto="fr"/>
-    <xacro:motor prefijo="tra_izq" corto="rl"/>
-    <xacro:motor prefijo="tra_der" corto="rr"/>
+    <xacro:motor prefijo="del_izq"/>
+    <xacro:motor prefijo="del_der"/>
+    <xacro:motor prefijo="tra_izq"/>
+    <xacro:motor prefijo="tra_der"/>
     <plugin filename="gz-sim-joint-state-publisher-system" name="gz::sim::systems::JointStatePublisher"/>
   </gazebo>
